Commit message: fix some bugs?

File: mr_description/urdf/g_module.urdf.xacro (robot description, xacro)
@@ -1,113 +1,184 @@
 <?xml version="1.0"?>
 <robot xmlns:xacro="http://www.ros.org/wiki/xacro">
+<xacro:property name="pi" value="3.1415926535897931" />
 <!--definition of default_inertial -->
-<xacro:macro name="g_module" params="parent name *origin">
-<!-- joint between base_link and Lockring_Link -->
+<xacro:macro name="G_module" params=" name parent *origin">
+<!-- joint between parent_link and palm _Link -->
   <joint name="${name}_joint_0" type="fixed" >
     <insert_block name="origin" />
     <parent link="${parent}" />
+    <child link="${name}_Link" />
+  </joint>
+  <link name="${name}_Link"/>
+<!-- joint between parent_link and palm _Link -->
+  <joint name="${name}_offset_joint" type="fixed" >
+    <origin xyz="0 0 0" rpy="${pi*0.5} 0 ${-pi*0.5}" />
+    <parent link="${name}_Link" />
     <child link="${name}_palm_link" />
   </joint>
+<!--the palm link-->
   <link name="${name}_palm_link">
+    <inertial>
+      <origin  xyz="-0.000330111921985683 0.0532067396112178 -0.00203994238779312"
+        rpy="0 0 0" />
+      <mass value="1.0043961075726" />
+      <inertia
+        ixx="0.00113334295507504"
+        ixy="8.90230328283654E-06"
+        ixz="-1.34473831837329E-06"
+        iyy="0.000914211060471031"
+        iyz="-6.54903141389812E-05"
+        izz="0.00129135037593152" />
+    </inertial>
     <visual>
-      <origin xyz="0 0 0" rpy="0 0 0" />
+      <origin
+        xyz="0 0 0"
+        rpy="0 0 0" />
       <geometry>
-        <mesh   filename="package://mr_description/meshes/g_palm_link.STL" />
+        <mesh filename="package://mr_description/meshes/palm_link.STL" />
       </geometry>
       <material  name="">
-        <color   rgba="0.1 0.1 0.1 1" />
-      </material>
-    </visual>
-    <collision>
-      <origin     xyz="0 0 0.028"    rpy="0 0 0" />
-      <geometry>
-<!--        <mesh  filename="package://mr_description/meshes/g_palm_link.STL" />-->
-	<cylinder radius="0.0425" length="0.056"/>
-      </geometry>
-    </collision>
-    <inertial>
-      <origin xyz="0.00425087794620391 -0.000341076549934847 0.0434713557042779" rpy="0 0 0" />
-      <mass value="0.566653469628951" />
-      <inertia
-        ixx="0.000498497223548746"
-        ixy="5.36329649188159E-07"
-        ixz="-4.07818737202901E-05"
-        iyy="0.000730511793998383"
-        iyz="-6.03266058697901E-06"
-        izz="0.000502182372067087" />
-    </inertial>
-  </link>
-  <joint  name="${name}_Joint"  type="prismatic">
-    <origin   xyz="0 0 0"    rpy="0 0 0" />
-    <parent   link="${name}_palm_link" />
-    <child   link="${name}_finger_link" />
-    <axis   xyz="-1 0 0" />
-    <limit    lower="0"  upper="0.06" effort="1" velocity="0.06" />
-<!--    <calibration   rising="1"   falling="1" />-->
-<!--    <dynamics    damping="1"    friction="1" />-->
-<!--    <safety_controller soft_upper="0.06" soft_lower="0" k_position="1" k_velocity="1" />-->
-  </joint>
-  <joint  name="${name}_Joint1"  type="prismatic">
-    <origin   xyz="0 0 0"    rpy="0 0 0" />
-    <parent    link="${name}_palm_link" />
-    <child    link="${name}_finger_link1" />
-    <axis   xyz="1 0 0" />
-    <limit  lower="0"  upper="0.06" effort="1" velocity="0.06" />
-<!--    <calibration  rising="1" />-->
-<!--    <dynamics  damping="1"  friction="1" />-->
-<!--    <safety_controller soft_upper="0.06" soft_lower="0" k_position="1" k_velocity="1" />-->
-  </joint>
-  <link  name="${name}_finger_link">
-    <visual>
-      <origin    xyz="0 0 0"     rpy="0 0 0" />
-      <geometry>
-        <mesh    filename="package://mr_description/meshes/g_finger_link.STL" />
-      </geometry>
-      <material    name="">
         <color rgba="0.1 0.1 0.1 1" />
       </material>
     </visual>
     <collision>
-      <origin   xyz="0 0 0"   rpy="0 0 0" />
+      <origin  xyz="0 0.065 0"  rpy="${pi*0.5} 0 0" />
+<!--      <origin  xyz="0 0 0"  rpy="0 0 0" />-->
       <geometry>
-        <mesh   filename="package://mr_description/meshes/g_finger_link.STL" />
+	<cylinder radius="0.05" length="0.12"/>
+<!--        <mesh filename="package://mr_description/meshes/palm_link.STL" />-->
       </geometry>
     </collision>
+  </link>
+  <!--the IModule_InLink Gazebo tag-->
+  <gazebo reference="${name}_palm_link">
+    <material>Gazebo/Black</material>
+  </gazebo>
+<!--  joint between the palm and the left finger-->
+  <joint name="${name}_Joint"  type="prismatic">
+    <origin xyz="0.038 0 0"  rpy="0 0 0" />
+    <parent link="${name}_palm_link" />
+    <child  link="${name}_finger_link_l" />
+    <axis   xyz="-1 0 0" />
+    <limit  lower="0"  upper="0.04" effort="10" velocity="0.02" />
+    <dynamics  damping="1" friction="1" />
+  </joint>
+   <!-- test reduction ratio-->
+  <transmission name="${name}_trans">
+    <type>transmission_interface/SimpleTransmission</type>
+    <joint name="${name}_Joint">
+      <hardwareInterface>PositionJointInterface</hardwareInterface>
+      <hardwareInterface>VelocityJointInterface</hardwareInterface>
+      <hardwareInterface>EffortJointInterface</hardwareInterface>
+    </joint>
+    <actuator name="${name}_motor">
+      <mechanicalReduction>400</mechanicalReduction>
+      <hardwareInterface>PositionJointInterface</hardwareInterface>
+      <hardwareInterface>VelocityJointInterface</hardwareInterface>
+      <hardwareInterface>EffortJointInterface</hardwareInterface>
+    </actuator>
+  </transmission>
+<!--  the left finger link-->
+  <link name="${name}_finger_link_l">
     <inertial>
-      <origin xyz="-0.0142537929479308 0.000230061402547915 0.123240994639791" rpy="0 0 0" />
-      <mass   value="0.0587979869361216" />
+      <origin  xyz="-0.053748 0.15337 2.2717E-07"  rpy="0 0 0" />
+      <mass   value="0.89853" />
       <inertia
-        ixx="4.06347072846223E-05" ixy="2.52194515964668E-08" ixz="9.16297919180235E-06"
-        iyy="4.29642140065611E-05" iyz="3.2622913893542E-08"  izz="9.72727638920999E-06" />
+        ixx="0.0023606"
+        ixy="-0.00017835"
+        ixz="4.9579E-09"
+        iyy="0.00087228"
+        iyz="-8.5058E-09"
+        izz="0.0018271" />
     </inertial>
-  </link>
-  <link  name="${name}_finger_link1">
     <visual>
-      <origin  xyz="0 0 0"  rpy="0 0 0" />
+      <origin  xyz="0 0 0" rpy="0 0 0" />
       <geometry>
-        <mesh filename="package://mr_description/meshes/g_finger_link1.STL" />
+        <mesh filename="package://mr_description/meshes/finger_link_l.STL" />
       </geometry>
-      <material    name="">
-        <color  rgba="0.1 0.1 0.1 1" />
+      <material name="">
+        <color  rgba="0.52941 0.54902 0.54902 1" />
       </material>
     </visual>
     <collision>
-      <origin    xyz="0 0 0"     rpy="0 0 0" />
+<!--      <origin xyz="-0.05 0.18 0" rpy="0 0 0" />-->
+      <origin xyz="0 0 0" rpy="0 0 0" />
       <geometry>
-        <mesh   filename="package://mr_description/meshes/g_finger_link1.STL" />
+<!--      	<box size="0.01 0.1 0.1"/>-->
+        <mesh filename="package://mr_description/meshes/finger_link_l.STL" />
       </geometry>
     </collision>
+  </link>
+  <!--the IModule_InLink Gazebo tag-->
+  <gazebo reference="${name}_finger_link_l">
+    <material>Gazebo/Black</material>
+  </gazebo>
+<!--  joint between the right finger and the palm-->
+  <joint  name="${name}_Joint1"  type="prismatic">
+    <origin  xyz="-0.038 0 0" rpy="0 0 0" />
+    <parent link="${name}_palm_link" />
+    <child  link="${name}_finger_link_r" />
+    <axis  xyz="1 0 0" />
+    <limit lower="0"  upper="0.04" effort="10" velocity="0.02" />
+    <dynamics   damping="1" friction="1" />
+  </joint>
+   <!-- test reduction ratio-->
+  <transmission name="${name}_trans1">
+    <type>transmission_interface/SimpleTransmission</type>
+    <joint name="${name}_Joint1">
+      <hardwareInterface>PositionJointInterface</hardwareInterface>
+      <hardwareInterface>VelocityJointInterface</hardwareInterface>
+      <hardwareInterface>EffortJointInterface</hardwareInterface>
+    </joint>
+    <actuator name="${name}_motor">
+      <mechanicalReduction>400</mechanicalReduction>
+      <hardwareInterface>PositionJointInterface</hardwareInterface>
+      <hardwareInterface>VelocityJointInterface</hardwareInterface>
+      <hardwareInterface>EffortJointInterface</hardwareInterface>
+    </actuator>
+  </transmission>
+<!-- the right finger link-->
+  <link name="${name}_finger_link_r">
     <inertial>
-      <origin xyz="0.0142537929479934 3.43816122645394E-05 0.123240994639808" rpy="0 0 0" />
-      <mass  value="0.0587979869361215" />
+      <origin   xyz="0.053748 0.15337 -2.2717E-07"  rpy="0 0 0" />
+      <mass    value="0.89853" />
       <inertia
-        ixx="4.06348713317454E-05"
-        ixy="4.84294028883443E-09"
-        ixz="-9.16297919179846E-06"
-        iyy="4.29642140065595E-05"
-        iyz="-7.56625401696782E-08"
-        izz="9.72744043633773E-06" />
+        ixx="0.0023606"
+        ixy="0.00017835"
+        ixz="4.9579E-09"
+        iyy="0.00087228"
+        iyz="8.5058E-09"
+        izz="0.0018271" />
     </inertial>
+    <visual>
+      <origin xyz="0 0 0" rpy="0 0 0" />
+      <geometry>
+        <mesh filename="package://mr_description/meshes/finger_link_r.STL" />
+      </geometry>
+      <material name="">
+        <color rgba="0.52941 0.54902 0.54902 1" />
+      </material>
+    </visual>
+    <collision>
+<!--      <origin xyz="0.05 0.18 0" rpy="0 0 0" />-->
+      <origin xyz="0 0 0" rpy="0 0 0" />
+      <geometry>
+<!--      	<box size="0.01 0.1 0.1"/>-->
+        <mesh filename="package://mr_description/meshes/finger_link_r.STL" />
+      </geometry>
+    </collision>
   </link>
+  <!--the IModule_InLink Gazebo tag-->
+  <gazebo reference="${name}_finger_link_r">
+    <material>Gazebo/Black</material>
+  </gazebo>
+<!--    joint between the palm link and the tcp-->
+  <joint name="${name}_tcp_joint" type="fixed">
+    <origin xyz="0 0.17836 0"  rpy="0 0 0" />
+    <parent link="${name}_palm_link" />
+    <child  link="${name}_tcp" />
+    <axis   xyz="0 0 0" />
+  </joint>
+  <link name="${name}_tcp" />
   </xacro:macro>
 </robot>
