Commit message: correct frames of mr5 and mr6

File: mr_description/robots/manipulator5d.urdf (robot description, URDF)
Before this commit: robot manipulator5d, 27 links, 26 joints
Links:
- removed link cl_100_85_connect_Link
- removed link i4_Link
- removed link i4_Offset_Link
- removed link i4_link
- removed link t5_Link
- removed link t5_Offset_Link
- removed link t5_link
- removed link tcp
- added link I4_Offset_Link, mass 0.80864; visual mesh filename=package://mr_description/meshes/i_link2.STL
- added link I4_link, mass 0.389080654611604; collision cylinder length=0.144 radius=0.0425; visual mesh filename=package://mr_description/meshes/i_link.STL
- added link T5_Offset_Link, mass 0.98367; collision cylinder length=0.125 radius=0.0425; visual mesh filename=package://mr_description/meshes/t_link2.STL
- added link T5_link, mass 0.832217409872162; collision cylinder length=0.052 radius=0.0425; visual mesh filename=package://mr_description/meshes/t_link.STL
Joints:
- removed joint i4_Joint
- removed joint i4_Offset_Joint
- removed joint i4_joint_0
- removed joint t5_Joint
- removed joint t5_Offset_Joint
- removed joint t5_joint_0
- removed joint tcp_fixed_joint
- added joint I4_Joint: type continuous, parent I4_link, child I4_Offset_Link, origin xyz=0 0 0.109 rpy=-8.5591E-29 0 0, axis 0 0 1, limit lower=-3.1416 upper=3.1416 effort=30 velocity=1.29
- added joint I4_Offset_Joint: type fixed, parent I4_Offset_Link, child T5_link, origin xyz=0 0 0.028 rpy=0 0 -1.57079632679
- added joint T5_Joint: type revolute, parent T5_link, child T5_Offset_Link, origin xyz=0.0123 0 0.131 rpy=0 -1.5708 3.1416, axis 0 0 1, limit lower=-2.09 upper=2.09 effort=28 velocity=2.09
- joint T2_Joint: axis 0 -1 0 -> 0 0 1; origin xyz= 0 0 0 rpy=4.7124 -1.2251E-16 3.1416 -> xyz= 0 0 0 rpy=0 3.1416 0
- joint T2_Lr_Joint_1: origin xyz=0 0 -0.1416 rpy=0 3.1416 0 -> xyz=0 0.1416 0 rpy=-1.5708 0 0
- joint T3_Joint: axis 0 0 -1 -> 0 0 1
- joint cl_fixed: child cl_100_85_connect_Link -> I4_link
- joint g6_joint_0: origin xyz=0 0 0 rpy=0 0 0 -> xyz=0.0825 0 -0.0123 rpy=0 1.5708 0; parent t5_Link -> T5_Offset_Link

File: mr_description/robots/manipulator6d.urdf (robot description, URDF)
Before this commit: robot ModuleManipulator, 27 links, 26 joints
Joints:
- joint T2_Joint: axis 0 -1 0 -> 0 0 1; origin xyz= 0 0 0 rpy=4.7124 -1.2251E-16 3.1416 -> xyz= 0 0 0 rpy=0 3.1416 0
- joint T2_Lr_Joint_1: origin xyz=0 0 -0.1416 rpy=0 3.1416 0 -> xyz=0 0.1416 0 rpy=-1.5708 0 0
- joint T4_Joint: axis 0 0 -1 -> 0 0 1
- joint g7_joint_0: origin xyz=0 0 0.0825 rpy=0 0 0 -> xyz=-0.0825 0 -0.0128 rpy=0 -1.5708 0
- joint t6_Joint: axis 1 0 0 -> 0 0 1; origin xyz=0 0 0.131 rpy=0 0 3.1416 -> xyz=0.0128 0 0.131 rpy=0 1.5708 0
